File: eagleman-vest-rev1/eagleman-vest-rev1.kicad_sch (KiCad schematic)
At the start: 93 parts, among them J10 Screw_Terminal_01x02, J11 Screw_Terminal_01x02, J2 Screw_Terminal_01x02, J3 Screw_Terminal_01x02, J4 Screw_Terminal_01x02, J5 Screw_Terminal_01x02, J6 Screw_Terminal_01x02, J7 Screw_Terminal_01x02, J8 Screw_Terminal_01x02, J9 Screw_Terminal_01x02, P1 USB_C_Plug_USB2.0, U1 ESP32-S3-WROOM-2, U10 DRV2605LDGSR, U11 DRV2605LDGSR, U12 DRV2605LDGSR, U13 DRV2605LDGSR, U14 DRV2605LDGSR, U15 DRV2605LDGSR, U16 DRV2605LDGSR, U2 AP1117-33, U3 TCA9548APWR, U4 TCA9548APWR, U7 DRV2605LDGSR, U8 DRV2605LDGSR, U9 DRV2605LDGSR

Commit message: started routing
Parts:
- removed D10, D11, D12, D13, D14, D5, D6, D7, D8, D9: LED, Capacitor_SMD:C_0603_1608Metric, symbol Device:LED
- removed R10, R11, R12, R13, R14, R15, R16, R7, R8, R9: 220, Capacitor_SMD:C_0603_1608Metric, symbol Device:R
- removed U1: ESP32-S3-WROOM-2, RF_Module:ESP32-S3-WROOM-2, symbol RF_Module:ESP32-S3-WROOM-2
- added C14: 100nF, Capacitor_SMD:C_0603_1608Metric, symbol Device:C
- added D31, D32, D33, D34, D35, D36, D37, D38, D39, D40: LED, Capacitor_SMD:C_0603_1608Metric, symbol Device:LED
- added J1, J17: Conn_01x08_Pin, Connector_PinHeader_2.54mm:PinHeader_1x08_P2.54mm_Vertical, symbol Connector:Conn_01x08_Pin
- added J12, J13: Conn_01x03_Pin, Connector_PinHeader_2.54mm:PinHeader_1x03_P2.54mm_Vertical, symbol Connector:Conn_01x03_Pin
- added J14: Conn_01x02_Pin, Connector_PinHeader_2.54mm:PinHeader_1x02_P2.54mm_Vertical, symbol Connector:Conn_01x02_Pin
- added J15: Conn_01x06_Pin, Connector_PinHeader_2.54mm:PinHeader_1x06_P2.54mm_Vertical, symbol Connector:Conn_01x06_Pin
- added J16: Conn_01x01_Pin, Connector_PinHeader_2.54mm:PinHeader_1x08_P2.54mm_Vertical, symbol Connector:Conn_01x01_Pin
- added J18: Conn_01x04_Pin, symbol Connector:Conn_01x04_Pin
- added R53, R54, R55, R56, R57, R58, R59, R60, R61, R62: 220, Capacitor_SMD:C_0603_1608Metric, symbol Device:R
- added R7: 10kΩ, PCM_JLCPCB:R_0402, symbol PCM_JLCPCB-Resistors:0402,10kΩ
- added SW1, SW2: SW_SPST, Button_Switch_SMD:SW_SPST_FSMSM, symbol Switch:SW_SPST
- added U5: ESP32-S3-WROOM-1, RF_Module:ESP32-S3-WROOM-1, symbol RF_Module:ESP32-S3-WROOM-1
- J10, J11, J2, J3, J4, J5, J6, J7, J8, J9: footprint (none) -> Connector_Phoenix_MC_HighVoltage:PhoenixContact_MCV_1,5_2-G-5.08_1x02_P5.08mm_Vertical
Connections:
- net GNDREF is gone; now on net GND: C1.2, C2.2, U2.1 (GND)
- net +3.3V: now also R7.1, U5.2 (3V3)
- net +5V: now also J15.3 (Pin_3)
- net GND: now also C14.2, D31.1 (K), D32.1 (K), D33.1 (K), D34.1 (K), D35.1 (K), D36.1 (K), D37.1 (K), D38.1 (K), D39.1 (K), D40.1 (K), J15.1 (Pin_1), SW1.1 (A), SW2.1 (A), U5.1 (GND), U5.40 (GND), U5.41 (GND)
- net GPIOEN: now also U5.18 (IO10)
- net f1-reset: now also U5.24 (IO47)
- net f2-reset: now also U5.25 (IO48)
- net scl: now also U5.17 (IO9)
- net sda: now also U5.12 (IO8)
- net at P1.A6 (D+): now also U5.14 (USB_D+)
- net at P1.A7 (D-): now also U5.13 (USB_D-)
- net f2-sc2: no longer names the net of U3.9 (SC2)
- net f2-sc2: now also J18.2 (Pin_2)
- net f2-sc3: no longer names the net of U3.11 (SC3)
- net f2-sc3: now also J18.4 (Pin_4)
- net f2-sc4: no longer names the net of U3.14 (SC4)
- net f2-sc4: now also J17.2 (Pin_2)
- net f2-sc5: no longer names the net of U3.16 (SC5)
- net f2-sc5: now also J17.4 (Pin_4)
- net f2-sc6: no longer names the net of U3.18 (SC6)
- net f2-sc6: now also J17.6 (Pin_6)
- net f2-sc7: no longer names the net of U3.20 (SC7)
- net f2-sc7: now also J17.8 (Pin_8)
- net f2-sd2: no longer names the net of U3.8 (SD2)
- net f2-sd2: now also J18.1 (Pin_1)
- net f2-sd3: no longer names the net of U3.10 (SD3)
- net f2-sd3: now also J18.3 (Pin_3)
- net f2-sd4: no longer names the net of U3.13 (SD4)
- net f2-sd4: now also J17.1 (Pin_1)
- net f2-sd5: no longer names the net of U3.15 (SD5)
- net f2-sd5: now also J17.3 (Pin_3)
- net f2-sd6: no longer names the net of U3.17 (SD6)
- net f2-sd6: now also J17.5 (Pin_5)
- net f2-sd7: no longer names the net of U3.19 (SD7)
- net f2-sd7: now also J17.7 (Pin_7)
- new net: D35.2 (A), R57.1
- new net: D33.2 (A), R55.1
- new net: J13.1 (Pin_1), U5.39 (IO1)
- new net: J13.2 (Pin_2), U5.38 (IO2)
- new net: J13.3 (Pin_3), U5.15 (IO3)
- new net: R55.2, U5.6 (IO6)
- new net: J15.6 (Pin_6), J16.1 (Pin_1)
- new net: D34.2 (A), R56.1
- new net: D36.2 (A), R58.1
- new net: J12.1 (Pin_1), U5.16 (IO46)
- new net: J12.2 (Pin_2), U5.26 (IO45)
- new net: J12.3 (Pin_3), U5.35 (IO42)
- new net: D37.2 (A), R59.1
- new net: R59.2, U5.19 (IO11)
- new net: D39.2 (A), R61.1
- new net: J14.2 (Pin_2), U5.10 (IO17)
- new net: J14.1 (Pin_1), U5.11 (IO18)
- new net: R60.2, U5.20 (IO12)
- new net: R61.2, U5.21 (IO13)
- new net: R62.2, U5.22 (IO14)
- new net: J1.8 (Pin_8), U5.23 (IO21)
- new net: J1.7 (Pin_7), U5.28 (IO35)
- new net: J1.6 (Pin_6), U5.29 (IO36)
- new net: J1.5 (Pin_5), U5.30 (IO37)
- new net: J1.4 (Pin_4), U5.31 (IO38)
- new net: J1.3 (Pin_3), U5.32 (IO39)
- new net: J1.2 (Pin_2), U5.33 (IO40)
- new net: J1.1 (Pin_1), U5.34 (IO41)
- new net: R54.2, U5.4 (IO4)
- new net: R53.2, U5.5 (IO5)
- new net: R56.2, U5.7 (IO7)
- new net: R57.2, U5.8 (IO15)
- new net: R58.2, U5.9 (IO16)
- new net: D40.2 (A), R62.1
- new net: D38.2 (A), R60.1
- new net: D32.2 (A), R54.1
- new net: D31.2 (A), R53.1
- new net BOOT_PIN: SW1.2 (B), U5.27 (IO0)
- new net EN_PIN: C14.1, R7.2, SW2.2 (B), U5.3 (EN)
- new net rx: J15.5 (Pin_5), U5.36 (RXD0)
- new net tx: J15.4 (Pin_4), U5.37 (TXD0)
Other:
- note removed: "shld i use this EN for the mux instead"
- moved on the sheet: C1, C2, C3, J10, J11, J2, J3, J4, J5, J6, J7, J8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

Commit message: i need help
Connections:
- net +5V: now also U14.1 (REG), U14.5 (EN); no longer U14.10 (VDD), U14.6 (VDD/NC)
- net GND: now also U14.3 (SDA), U14.7 (OUT+); no longer U14.4 (IN/TRIG), U14.8 (GND)
- net GPIOEN: now also U14.6 (VDD/NC); no longer U14.5 (EN)
- net f1-sc4: now also U14.9 (OUT-); no longer U14.2 (SCL)
- net f1-sd4: now also U14.8 (GND); no longer U14.3 (SDA)
- net at J9.1 (Pin_1): now also U14.2 (SCL); no longer U14.9 (OUT-)
- net at J9.2 (Pin_2): now also U14.4 (IN/TRIG); no longer U14.7 (OUT+)
- net at C10.1: now also U14.10 (VDD); no longer U14.1 (REG)
Changed lines of the file:
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@@
 		(lib_id "DRV2605LDGSR:DRV2605LDGSR")
 		(at 120.65 156.21 0)
+		(mirror y)
 		(unit 1)
 		(exclude_from_sim no)
@@
 		(on_board yes)
 		(dnp no)
-		(fields_autoplaced yes)
 		(property "Reference" "U14"
 			(at 120.65 143.51 0)
@@
 		)
 		(property "Datasheet" "https://item.szlcsc.com/202966.html"
-			(at 118.364 156.083 0)
+			(at 122.936 156.083 0)
 			(effects
 				(font

Commit message: updated routing and lowered density a little bit
Parts:
- removed J12, J13: Conn_01x03_Pin, Connector_PinHeader_2.54mm:PinHeader_1x03_P2.54mm_Vertical, symbol Connector:Conn_01x03_Pin
- removed R4, R6: 4.7kΩ, PCM_JLCPCB:R_0402, symbol PCM_JLCPCB-Resistors:0402,4.7kΩ
- added J19: Conn_01x06_Pin, Connector_PinHeader_2.54mm:PinHeader_1x06_P2.54mm_Vertical, symbol Connector:Conn_01x06_Pin
- C10, C11, C12, C13, C24, C25, C27, C29, C3, C30, C32, C33, C35, C36, C4, C5, C6, C7, C8, C9: footprint PCM_JLCPCB:C_0402 -> Capacitor_SMD:C_0603_1608Metric
- J16: footprint Connector_PinHeader_2.54mm:PinHeader_1x08_P2.54mm_Vertical -> Connector_PinHeader_1.27mm:PinHeader_1x01_P1.27mm_Vertical
- J17: footprint Connector_PinHeader_2.54mm:PinHeader_1x08_P2.54mm_Vertical -> Connector_PinHeader_1.27mm:PinHeader_1x08_P1.27mm_Vertical
- J18: footprint (none) -> Connector_PinHeader_1.27mm:PinHeader_1x04_P1.27mm_Vertical
- R1, R2: footprint PCM_JLCPCB:R_0805 -> Capacitor_SMD:C_0603_1608Metric
- R17, R18, R19, R20, R21, R22, R23, R24, R25, R26, R27, R28, R29, R3, R30, R31, R32, R33, R34, R35, R36, R5, R7: footprint PCM_JLCPCB:R_0402 -> Capacitor_SMD:C_0603_1608Metric
- U14: footprint TCA9548APWR:driver_footprint_maybe -> DRV2605:SOP50P490X110-10N
Connections:
- net +5V: now also U14.10 (VDD), U14.6 (VDD/NC); no longer U14.1 (REG), U14.5 (EN)
- net GND: now also U14.4 (IN/TRIG), U14.8 (GND), U15.4 (IN/TRIG); no longer U14.3 (SDA), U14.7 (OUT+)
- net GPIOEN: now also U14.5 (EN); no longer U14.6 (VDD/NC)
- net f1-sc4: now also U14.2 (SCL); no longer U14.9 (OUT-)
- net f1-sd4: now also U14.3 (SDA); no longer U14.8 (GND)
- net at J9.1 (Pin_1): now also U14.9 (OUT-); no longer U14.2 (SCL)
- net at J9.2 (Pin_2): now also U14.7 (OUT+); no longer U14.4 (IN/TRIG)
- net p1: now reaches U5.39 (IO1)
- net p1: now also J19.6 (Pin_6)
- net p2: now reaches U5.38 (IO2)
- net p2: now also J19.5 (Pin_5)
- net p3: now reaches U5.15 (IO3)
- net p3: now also J19.4 (Pin_4)
- net at C10.1: now also U14.1 (REG); no longer U14.10 (VDD)
- net p46: now reaches U5.16 (IO46)
- net p46: now also J19.3 (Pin_3)
- net p45: now reaches U5.26 (IO45)
- net p45: now also J19.2 (Pin_2)
- net p42: now reaches U5.35 (IO42)
- net p42: now also J19.1 (Pin_1)
Other:
- moved on the sheet: J17, J18
